File: 180V DC Driver/180V_DC_Driver/180V_DC_Driver_3mm.kicad_pcb (KiCad board)
At the start: 2 copper layers, 195 x 112 mm, 16 parts, among them J1 AC_In, J2 DC_Out, J3 Conn_01x02_Socket, J4 Conn_01x01_Socket, Q1 IRFP460PBF

Commit message: c2.06
Parts:
- moved J2 15.2 mm to (112.0, 103.5)
- moved D2 15.0 mm to (97.0, 103.9)
