File: 180V DC Driver/180V_DC_Driver/180V_DC_Driver.kicad_pcb (KiCad board)
At the start: 2 copper layers, 195 x 112 mm, 16 parts, among them J1 AC_In, J2 DC_Out, J3 Conn_01x02_Socket, J4 Conn_01x01_Socket, Q1 IRFP460PBF

Commit message: c1806
Routing:
- net Net-(BR1-+): track 254.8 -> 249.2 mm

Commit message: c22.06
Parts:
- added RV1: Varistor, Capacitor_THT:C_Disc_D10.5mm_W5.0mm_P5.00mm, F.Cu at (69.0, 30.0)
Routing:
- net Net-(PS1-AC_1): track 21.6 -> 29.6 mm
- net Net-(BR1-~_1): track 132.5 -> 138.5 mm
