File: 180V DC Driver/180V_DC_Driver/180V_DC_Driver_down.kicad_pcb (KiCad board)
At the start: 2 copper layers, 194 x 112 mm, 18 parts, among them J1 AC_In, J2 DC_Out, J3 Conn_01x02_Socket, J4 Conn_01x01_Socket, Q1 IRFP460PBF

Commit message: c28.06
Parts:
- moved J2 108.7 mm to (96.8, 103.5), turned to -90 degrees
- moved D2 81.5 mm to (112.0, 103.5), turned to -90 degrees
- moved J4 71.2 mm to (135.0, 116.0), turned to 0 degrees
- moved R3 67.1 mm to (144.9, 116.0), turned to 0 degrees
- moved Q1 44.9 mm to (144.6, 104.8), turned to 0 degrees
- moved C5 23.5 mm to (126.0, 78.0)
- moved C1 23.3 mm to (155.0, 87.1)
- moved R1 23.0 mm to (191.0, 81.1)
- moved C3 22.5 mm to (176.0, 87.8)
- moved C4 22.2 mm to (80.0, 78.3)
Routing:
- net Net-(BR1--): track 242.8 -> 292.4 mm
- net Net-(BR1-+): track 254.3 -> 251.1 mm
Other:
- board size 194 x 112 mm -> 195 x 112 mm
- board text removed: "MEM-R 180V DC DRIVER"
